File: lab4/exercise1/exercise1.kicad_sch (KiCad schematic)
At the start: 6 parts, among them SW1 SW_SPDT

Commit message: adding lab 4 changes with pcb
Parts:
- C1: footprint (none) -> Capacitor_THT:C_Radial_D5.0mm_H5.0mm_P2.00mm
- D1: footprint (none) -> LED_THT:LED_D5.0mm
- R1, R2: footprint (none) -> Resistor_THT:R_Axial_DIN0516_L15.5mm_D5.0mm_P20.32mm_Horizontal
- SW1: footprint (none) -> Button_Switch_THT:SW_E-Switch_EG1224_SPDT_Angled
- V1: footprint (none) -> Connector_JST:JST_PH_B2B-PH-K_1x02_P2.00mm_Vertical
Changed lines of the file:
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@@
       (effects (font (size 1.27 1.27)) (justify right))
     )
-    (property "Footprint" "" (id 2) (at 99.06 116.84 0)
+    (property "Footprint" "LED_THT:LED_D5.0mm" (id 2) (at 99.06 116.84 0)
       (effects (font (size 1.27 1.27)) hide)
     )
@@
       (effects (font (size 1.27 1.27)) (justify left))
     )
-    (property "Footprint" "" (id 2) (at 79.7052 109.22 0)
+    (property "Footprint" "Capacitor_THT:C_Radial_D5.0mm_H5.0mm_P2.00mm" (id 2) (at 79.7052 109.22 0)
       (effects (font (size 1.27 1.27)) hide)
     )
@@
     (property "Reference" "V1" (id 0) (at 40.64 99.06 0))
     (property "Value" "9V" (id 1) (at 40.64 101.6 0))
-    (property "Footprint" "" (id 2) (at 43.18 100.33 0)
+    (property "Footprint" "Connector_JST:JST_PH_B2B-PH-K_1x02_P2.00mm_Vertical" (id 2) (at 43.18 100.33 0)
       (effects (font (size 1.27 1.27)) hide)
     )
@@
       (effects (font (size 1.27 1.27)) hide)
     )
-    (property "Footprint" "" (id 2) (at 71.12 86.36 0)
+    (property "Footprint" "Button_Switch_THT:SW_E-Switch_EG1224_SPDT_Angled" (id 2) (at 71.12 86.36 0)
       (effects (font (size 1.27 1.27)) hide)
     )
@@
       (effects (font (size 1.27 1.27)) (justify left))
     )
-    (property "Footprint" "" (id 2) (at 97.282 100.33 90)
+    (property "Footprint" "Resistor_THT:R_Axial_DIN0516_L15.5mm_D5.0mm_P20.32mm_Horizontal" (id 2) (at 97.282 100.33 90)
       (effects (font (size 1.27 1.27)) hide)
     )
@@
     (property "Reference" "R2" (id 0) (at 52.07 80.01 90))
     (property "Value" "2.2K" (id 1) (at 52.07 82.55 90))
-    (property "Footprint" "" (id 2) (at 52.07 84.582 90)
+    (property "Footprint" "Resistor_THT:R_Axial_DIN0516_L15.5mm_D5.0mm_P20.32mm_Horizontal" (id 2) (at 52.07 84.582 90)
       (effects (font (size 1.27 1.27)) hide)
     )
@@
   (symbol_instances
     (path "/5bfa2a17-0e72-4c2f-981b-7240492221ca"
-      (reference "C1") (unit 1) (value "4.7uF") (footprint "")
+      (reference "C1") (unit 1) (value "4.7uF") (footprint "Capacitor_THT:C_Radial_D5.0mm_H5.0mm_P2.00mm")
     )
     (path "/12dfbf8e-f8e3-43af-829f-491c6d54a78b"
-      (reference "D1") (unit 1) (value "LED") (footprint "")
+      (reference "D1") (unit 1) (value "LED") (footprint "LED_THT:LED_D5.0mm")
     )
     (path "/db77911e-892d-47d1-b571-5d907c83a1b4"
-      (reference "R1") (unit 1) (value "20K") (footprint "")
+      (reference "R1") (unit 1) (value "20K") (footprint "Resistor_THT:R_Axial_DIN0516_L15.5mm_D5.0mm_P20.32mm_Horizontal")
     )
     (path "/e0b0a0bf-7cf5-4499-a097-64e828a059cb"
-      (reference "R2") (unit 1) (value "2.2K") (footprint "")
+      (reference "R2") (unit 1) (value "2.2K") (footprint "Resistor_THT:R_Axial_DIN0516_L15.5mm_D5.0mm_P20.32mm_Horizontal")
     )
     (path "/b2ba34f8-8978-4db5-a9e9-6715e671d36b"
-      (reference "SW1") (unit 1) (value "SW_SPDT") (footprint "")
+      (reference "SW1") (unit 1) (value "SW_SPDT") (footprint "Button_Switch_THT:SW_E-Switch_EG1224_SPDT_Angled")
     )
     (path "/678d646f-b849-4168-95dc-d01b8a21c616"
-      (reference "V1") (unit 1) (value "9V") (footprint "")
+      (reference "V1") (unit 1) (value "9V") (footprint "Connector_JST:JST_PH_B2B-PH-K_1x02_P2.00mm_Vertical")
     )
   )
