File: lab4/exercise2/exercise2.kicad_sch (KiCad schematic)
At the start: 10 parts, among them J1 J1, U1 U1

Commit message: adding lab 4 changes with pcb
Parts:
- C1: footprint (none) -> Capacitor_Tantalum_SMD:CP_EIA-3216-18_Kemet-A_Pad1.58x1.35mm_HandSolder
- C2: footprint (none) -> Capacitor_SMD:C_0805_2012Metric_Pad1.18x1.45mm_HandSolder
- D1, D2: footprint (none) -> LED_SMD:LED_1206_3216Metric_Pad1.42x1.75mm_HandSolder
- J1: footprint (none) -> TerminalBlock:TerminalBlock_bornier-2_P5.08mm
- R1, R2, R3, R4: footprint (none) -> Resistor_SMD:R_0805_2012Metric_Pad1.20x1.40mm_HandSolder
- U1: footprint Package_SO:SOIC-8_3.9x4.9mm_P1.27mm -> Package_SO:SOIC-8-1EP_3.9x4.9mm_P1.27mm_EP2.29x3mm
Changed lines of the file:
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@@
   (symbol (lib_name "GND_1") (lib_id "power:GND") (at 124.46 147.32 0) (unit 1)
     (in_bom yes) (on_board yes) (fields_autoplaced)
-    (property "Reference" "#PWR?" (id 0) (at 124.46 153.67 0)
+    (property "Reference" "#PWR0101" (id 0) (at 124.46 153.67 0)
       (effects (font (size 1.27 1.27)) hide)
     )
@@
       (effects (font (size 1.27 1.27)) (justify right))
     )
-    (property "Footprint" "" (id 2) (at 189.23 81.28 0)
+    (property "Footprint" "LED_SMD:LED_1206_3216Metric_Pad1.42x1.75mm_HandSolder" (id 2) (at 189.23 81.28 0)
       (effects (font (size 1.27 1.27)) hide)
     )
@@
       (effects (font (size 1.27 1.27)) (justify left))
     )
-    (property "Footprint" "" (id 2) (at 70.612 82.55 90)
+    (property "Footprint" "Resistor_SMD:R_0805_2012Metric_Pad1.20x1.40mm_HandSolder" (id 2) (at 70.612 82.55 90)
       (effects (font (size 1.27 1.27)) hide)
     )
@@
     )
     (property "Value" "J1" (id 1) (at 133.35 74.93 90))
-    (property "Footprint" "" (id 2) (at 127 69.85 0)
+    (property "Footprint" "TerminalBlock:TerminalBlock_bornier-2_P5.08mm" (id 2) (at 127 69.85 0)
       (effects (font (size 1.27 1.27)) hide)
     )
@@
       (effects (font (size 1.27 1.27)) (justify left))
     )
-    (property "Footprint" "" (id 2) (at 70.612 113.03 90)
+    (property "Footprint" "Resistor_SMD:R_0805_2012Metric_Pad1.20x1.40mm_HandSolder" (id 2) (at 70.612 113.03 90)
       (effects (font (size 1.27 1.27)) hide)
     )
@@
       (effects (font (size 1.27 1.27)) (justify right))
     )
-    (property "Footprint" "" (id 2) (at 189.23 137.16 0)
+    (property "Footprint" "LED_SMD:LED_1206_3216Metric_Pad1.42x1.75mm_HandSolder" (id 2) (at 189.23 137.16 0)
       (effects (font (size 1.27 1.27)) hide)
     )
@@
       (effects (font (size 1.27 1.27)) (justify left))
     )
-    (property "Footprint" "" (id 2) (at 187.452 114.3 90)
+    (property "Footprint" "Resistor_SMD:R_0805_2012Metric_Pad1.20x1.40mm_HandSolder" (id 2) (at 187.452 114.3 90)
       (effects (font (size 1.27 1.27)) hide)
     )
@@
   (symbol (lib_name "+9V_1") (lib_id "power:+9V") (at 127 67.31 0) (mirror y) (unit 1)
     (in_bom yes) (on_board yes) (fields_autoplaced)
-    (property "Reference" "#PWR?" (id 0) (at 127 71.12 0)
+    (property "Reference" "#PWR0105" (id 0) (at 127 71.12 0)
       (effects (font (size 1.27 1.27)) hide)
     )
@@
       (effects (font (size 1.27 1.27)) (justify left) hide)
     )
-    (property "Footprint" "Package_SO:SOIC-8_3.9x4.9mm_P1.27mm" (id 2) (at 156.21 114.3 0)
+    (property "Footprint" "Package_SO:SOIC-8-1EP_3.9x4.9mm_P1.27mm_EP2.29x3mm" (id 2) (at 156.21 114.3 0)
       (effects (font (size 1.27 1.27)) hide)
     )
@@
       (effects (font (size 1.27 1.27)) (justify left))
     )
-    (property "Footprint" "" (id 2) (at 73.3552 140.97 0)
+    (property "Footprint" "Capacitor_Tantalum_SMD:CP_EIA-3216-18_Kemet-A_Pad1.58x1.35mm_HandSolder" (id 2) (at 73.3552 140.97 0)
       (effects (font (size 1.27 1.27)) hide)
     )
@@
   (symbol (lib_id "power:+9V") (at 72.39 78.74 0) (unit 1)
     (in_bom yes) (on_board yes) (fields_autoplaced)
-    (property "Reference" "#PWR?" (id 0) (at 72.39 82.55 0)
+    (property "Reference" "#PWR0104" (id 0) (at 72.39 82.55 0)
       (effects (font (size 1.27 1.27)) hide)
     )
@@
   (symbol (lib_name "+9V_3") (lib_id "power:+9V") (at 189.23 77.47 0) (unit 1)
     (in_bom yes) (on_board yes) (fields_autoplaced)
-    (property "Reference" "#PWR?" (id 0) (at 189.23 81.28 0)
+    (property "Reference" "#PWR0103" (id 0) (at 189.23 81.28 0)
       (effects (font (size 1.27 1.27)) hide)
     )
@@
   (symbol (lib_id "power:GND") (at 129.54 67.31 0) (mirror x) (unit 1)
     (in_bom yes) (on_board yes)
-    (property "Reference" "#PWR?" (id 0) (at 129.54 60.96 0)
+    (property "Reference" "#PWR0106" (id 0) (at 129.54 60.96 0)
       (effects (font (size 1.27 1.27)) hide)
     )
@@
       (effects (font (size 1.27 1.27)) (justify left))
     )
-    (property "Footprint" "" (id 2) (at 187.452 97.79 90)
+    (property "Footprint" "Resistor_SMD:R_0805_2012Metric_Pad1.20x1.40mm_HandSolder" (id 2) (at 187.452 97.79 90)
       (effects (font (size 1.27 1.27)) hide)
     )
@@
   (symbol (lib_name "+9V_2") (lib_id "power:+9V") (at 134.62 86.36 0) (unit 1)
     (in_bom yes) (on_board yes) (fields_autoplaced)
-    (property "Reference" "#PWR?" (id 0) (at 134.62 90.17 0)
+    (property "Reference" "#PWR0102" (id 0) (at 134.62 90.17 0)
       (effects (font (size 1.27 1.27)) hide)
     )
@@
       (effects (font (size 1.27 1.27)) (justify left))
     )
-    (property "Footprint" "" (id 2) (at 97.4852 127 0)
+    (property "Footprint" "Capacitor_SMD:C_0805_2012Metric_Pad1.18x1.45mm_HandSolder" (id 2) (at 97.4852 127 0)
       (effects (font (size 1.27 1.27)) hide)
     )
@@
   (symbol_instances
     (path "/0603331a-9711-4b30-b368-e7d7f1b8e5c5"
-      (reference "#PWR?") (unit 1) (value "GND") (footprint "")
+      (reference "#PWR0101") (unit 1) (value "GND") (footprint "")
+    )
+    (path "/e7004b57-fc30-4a94-a437-4aed7a7a62b1"
+      (reference "#PWR0102") (unit 1) (value "+9V") (footprint "")
+    )
+    (path "/c7abd33c-6157-4faf-8919-aaad3acd9c28"
+      (reference "#PWR0103") (unit 1) (value "+9V") (footprint "")
+    )
+    (path "/a27256e5-3667-4cd0-9ae8-a60c7f5f738a"
+      (reference "#PWR0104") (unit 1) (value "+9V") (footprint "")
     )
     (path "/5e52cb2e-a760-4fe6-bd1a-89cd60fa49f3"
-      (reference "#PWR?") (unit 1) (value "+9V") (footprint "")
-    )
-    (path "/a27256e5-3667-4cd0-9ae8-a60c7f5f738a"
-      (reference "#PWR?") (unit 1) (value "+9V") (footprint "")
-    )
-    (path "/c7abd33c-6157-4faf-8919-aaad3acd9c28"
-      (reference "#PWR?") (unit 1) (value "+9V") (footprint "")
+      (reference "#PWR0105") (unit 1) (value "+9V") (footprint "")
     )
     (path "/d44692b0-bf26-4d33-a2ff-bff68de7d299"
-      (reference "#PWR?") (unit 1) (value "GND") (footprint "")
-    )
-    (path "/e7004b57-fc30-4a94-a437-4aed7a7a62b1"
-      (reference "#PWR?") (unit 1) (value "+9V") (footprint "")
+      (reference "#PWR0106") (unit 1) (value "GND") (footprint "")
     )
     (path "/6e9e1a97-4607-4800-a99b-3779130c6487"
-      (reference "C1") (unit 1) (value "10uF") (footprint "")
+      (reference "C1") (unit 1) (value "10uF") (footprint "Capacitor_Tantalum_SMD:CP_EIA-3216-18_Kemet-A_Pad1.58x1.35mm_HandSolder")
     )
     (path "/fc9f1e48-47cb-4118-be65-100c647e414c"
-      (reference "C2") (unit 1) (value "0.01uF") (footprint "")
+      (reference "C2") (unit 1) (value "0.01uF") (footprint "Capacitor_SMD:C_0805_2012Metric_Pad1.18x1.45mm_HandSolder")
     )
     (path "/0ee6c829-77c2-4e2e-a787-a5e251736abd"
-      (reference "D1") (unit 1) (value "LED") (footprint "")
+      (reference "D1") (unit 1) (value "LED") (footprint "LED_SMD:LED_1206_3216Metric_Pad1.42x1.75mm_HandSolder")
     )
     (path "/4a5de5b5-666f-4ad1-836e-53b3d3b2cfdd"
-      (reference "D2") (unit 1) (value "LED") (footprint "")
+      (reference "D2") (unit 1) (value "LED") (footprint "LED_SMD:LED_1206_3216Metric_Pad1.42x1.75mm_HandSolder")
     )
     (path "/28057500-a34f-4141-89f5-1d6fd754d7fd"
-      (reference "J1") (unit 1) (value "J1") (footprint "")
+      (reference "J1") (unit 1) (value "J1") (footprint "TerminalBlock:TerminalBlock_bornier-2_P5.08mm")
     )
     (path "/21d83f80-6498-4aac-bb97-566c90b837b7"
-      (reference "R1") (unit 1) (value "1k") (footprint "")
+      (reference "R1") (unit 1) (value "1k") (footprint "Resistor_SMD:R_0805_2012Metric_Pad1.20x1.40mm_HandSolder")
     )
     (path "/2de06ac0-17f0-4015-93ff-3027f8fa0e4d"
-      (reference "R2") (unit 1) (value "10k") (footprint "")
+      (reference "R2") (unit 1) (value "10k") (footprint "Resistor_SMD:R_0805_2012Metric_Pad1.20x1.40mm_HandSolder")
     )
     (path "/d5423132-27ef-46cc-84de-7ac7c84efdab"
-      (reference "R3") (unit 1) (value "1k") (footprint "")
+      (reference "R3") (unit 1) (value "1k") (footprint "Resistor_SMD:R_0805_2012Metric_Pad1.20x1.40mm_HandSolder")
     )
     (path "/5bbce860-8fb3-4aee-9208-39f67f95136e"
-      (reference "R4") (unit 1) (value "1k") (footprint "")
+      (reference "R4") (unit 1) (value "1k") (footprint "Resistor_SMD:R_0805_2012Metric_Pad1.20x1.40mm_HandSolder")
     )
     (path "/6403c71a-21e2-453f-a4b6-29f5b52ee83c"
-      (reference "U1") (unit 1) (value "U1") (footprint "Package_SO:SOIC-8_3.9x4.9mm_P1.27mm")
-    )
-  )
+      (reference "U1") (unit 1) (value "U1") (footprint "Package_SO:SOIC-8-1EP_3.9x4.9mm_P1.27mm_EP2.29x3mm")
+    )
+  )
